Commit message: added color gradient

File: test/index_urdf.urdf (robot description, URDF)
Before this commit: robot urdf_rom_visualizer/index_urdf, 5 links, 5 joints
Joints:
- joint ima_joint: origin xyz=-0.030085 -0.0405 0.11024 rpy=-1.5708 -1.4573 -3.1416 -> xyz=0 0 0 rpy=-1.5708 -1.4573 -3.1416

File: test/thumb_urdf.urdf (robot description, URDF)
Before this commit: robot urdf_rom_visualizer/urdf, 6 links, 6 joints
Joints:
- joint tcf_joint: origin xyz=-0.03245 -0.0217 0.0495 rpy=0 0 0 -> xyz=0 0 0 rpy=0 0 0
